File: rs-probe.kicad_sch (KiCad schematic)
At the start: 98 parts, among them J1 USB_C_Receptacle_USB2.0, J10 Conn_01x01, J11 Conn_01x01, J2 Castellated Vias, J3 Castellated Vias, J4 Castellated Vias, J5 tag-connect-swd, J6 Conn_01x01, J7 Conn_01x01, J8 Conn_01x01, J9 Conn_01x01, Q1 NTZD3155C or CMLDM3757-TR-PBF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, SW1 EVQ-P2002W, T1 Tab, T2 Tab, U1 74LVC1T45GM,115, U10 74LVC1T45GM,115, U11 74LVC1T45GM,115, U12 NCP133AMXADJTCG, U13 NCP133AMXADJTCG, U14 NCP133AMXADJTCG, U2 74LVC1T45GM,115, U3 W25Q8, U4 NUF8401MNT4G, U5 CortexDebug, U6 RP2040, U7 NUF2042XV6T1G, U8 74LVC1T45GM,115, U9 74LVC1T45GM,115, X1 12 MHz

Commit message: Modification for BillMock-HW on-site programming
Parts:
- removed J2: Castellated Vias, connectors:1x9_1.5mm_castellated, symbol Connector_Generic:Conn_01x09
- removed J3: Castellated Vias, connectors:1x2_1.5mm_castellated, symbol Connector_Generic:Conn_01x02
- added C31: 0.1u, passive:C_0402, symbol Device:C_Small
- added J12: Conn_01x01, connectors:pad_1.5x2.0mm, symbol Connector_Generic:Conn_01x01
- added J2: Conn_02x05_Odd_Even, tc-custom:TC2050-ProbeMod, symbol Connector_Generic:Conn_02x05_Odd_Even
- added R30: 0Ω, passive:R_0402, symbol Device:R_Small
- added R31: 1k, passive:R_0402, symbol Device:R_Small
- added R32, R33: 3.3kΩ 1608, passive:R_0603, symbol Device:R_Small
- added SW2: TS-1145A-C-B, Button_Switch_SMD_Extended:SW_SPST_TS-1145A, symbol Switch:SW_Push
- added SYM1: SYM_Arrow45_Normal, Symbol_Extended:LamudaEE-12.3x7.6mm, symbol Graphic:SYM_Arrow45_Normal
- added U15: FM24V02A-GTR, Package_SO:SOIC-8_3.9x4.9mm_P1.27mm, symbol Memory_NVRAM:FM24C64B
- C1, C10, C11, C12, C13, C14, C15, C16, C17, C18, C19, C20, C22, C23, C28, C5, C7, C8, C9: LCSC C56392 -> C307331; MFPN (none) -> CL05B104KB54PNC
- C2, C21, C24, C25, C26, C27, C29, C3, C30, C4, C6: LCSC C77002 -> C170151; MFPN (none) -> CL05A225KO5NQNC
- D1: Alternative (none) -> C427425, C458749; LCSC C427425, C458749 -> C458749
- D2, D3: Alternative (none) -> SBA0520Q or similar; LCSC (none) -> C145312; MFPN SBA0520Q or similar -> VSKY05401006-G4-08
- F1: MFPN MF-FSMF050X-2 -> MF-FSMF050X-2
- FB1: LCSC (none) -> C76886
- J1: JLCPCB Position Offset (none) -> 0,1.4
- J4, TP1, TP2, TP3, TP4: now left out of the parts list
- Q1: value NTZD3155C or CMLDM3757-TR-PBFREE or DMC2400UV-7 or DMG1016VQ-7 -> NTZD3155C; Alternative (none) -> C895156, C236117, C3280275, C177025, C2940616; JLCPCB Rotation Offset (none) -> 270; LCSC C895156, C236117, C3280275, C177025, C2940616 -> C895156; MFPN NTZD3155C or CMLDM3757-TR-PBFREE or DMC2400UV-7 or DMG1016V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 -> NTZD3155C
- R1, R13, R15, R28: LCSC C409673 -> C26957
- R11, R12, R14, R16, R19, R21, R27, R9: LCSC C144757 -> C25792
- R17, R2, R5, R6, R7: LCSC C106235 -> C11702
- R20: LCSC (none) -> C25905
- R25: LCSC C409673 -> C25756
- R29, R3, R4, R8: LCSC C105872 -> C25905
- SW1: value EVQ-P2002W -> TS-1145A-C-B; footprint Button_Switch_SMD:SW_SPST_EVQP2 -> Button_Switch_SMD_Extended:SW_SPST_TS-1145A; Alternative (none) -> Original : C79148, C713481; LCSC C79148, C713481 -> C465998; MFPN EVQ-P2002W -> TS-1145A-C-B
- U1, U10, U11, U2, U8, U9: value 74LVC1T45GM,115 -> 74LVC1T45FZ4-7; footprint Package_TO_SOT_SMD:SOT-886 -> Package_DFN_QFN_Extended:X2-DFN1410-6; JLCPCB Rotation Offset (none) -> 270; LCSC C548481, C548480, C548479 -> C150482; MFPN 74LVC1T45GM,115 -> 74LVC1T45FZ4-7
- U12, U13, U14, U4: JLCPCB Rotation Offset (none) -> 270
- U3: value W25Q8 -> IS25WP016D-JULE-TR; Alternative (none) -> C2976734, C2759920, C2983691, C559220, C394861; LCSC C2063555, C2759920, C2983691, C559220, C394861 -> C2976734; MFPN W25Q80DVUXIE -> IS25WP016D
- U5: Alternative (none) -> C2935458, C448647; JLCPCB Rotation Offset (none) -> 270; LCSC C2935458, C150517, C920815 -> C448647; MFPN FTSH-105-01-L-DV-K -> FTSH-105-01-L-DV-K-TR
- X1: Alternative (none) -> C255991, C2681259, C3034288, C2901596; LCSC C255991, C2681259, C3034288, C2901596 -> C255991; MFPN ISM95-3251AH-12.000MHZ -> ISM95-3251AH-12.000MHZ
Connections:
- net +3.3V: now also C31.1, R32.2, R33.2, U15.8 (VDD)
- net GND: now also C31.2, J2.7 (Pin_7), SW2.1, U15.1 (A0), U15.2 (A1), U15.3 (A2), U15.4 (VSS), U15.7 (WP)
- net GPIO1: now also J12.1 (Pin_1), R31.1
- net T_GNDDetect: now also J2.8 (Pin_8)
- net T_SWDCLK_JCLK: now also J2.4 (Pin_4)
- net T_SWDIO_TMS: now also J2.3 (Pin_3)
- net T_SWO_TDO: now also J2.1 (Pin_1)
- net T_TDI: now also J2.2 (Pin_2)
- net T_VCC: now also R30.2
- net T_VCP_RX: now also J2.9 (Pin_9)
- net T_VCP_TX: now also J2.10 (Pin_10)
- net T_~{RESET}: now also J2.5 (Pin_5)
- net FRAM_SDA: now reaches U6.17 (GPIO14)
- net FRAM_SDA: now also R32.1, U15.5 (SDA)
- net FRAM_SCL: now reaches U6.18 (GPIO15)
- net FRAM_SCL: now also R33.1, U15.6 (SCL)
- new net: R31.2, SW2.2
- new net T_VCC_PROTECT: J2.6 (Pin_6), R30.1
- no-connect marks 11 -> 9
Other:
- note added: "Additional tact switch"
- note added: "Modified Part - FRAM addiction Store data such as flash count or affected target device ID"
- note added: "Original Designed by: Emil Fresk | Twitter / Github: @korken89 Link: https://github.com/probe-rs/rs-probe Modified by : Jinwoo PArk (github.com/pmnxis)"
- note added: "Pen type SWD TC-2030 assembly for BillMock-HW"
- note removed: "Designed by: Emil Fresk Twitter / Github: @korken89 Link: https://github.com/probe-rs/rs-probe"
- title: The Rusty Probe -> The Rusty Probe (HandyJig Mod)

Commit message: Fabricated on JLCPCB (not tested yet)
Parts:
- added TH1, TH2, TH3, TH4: Tooling Hole, symbol Connector_Generic:Conn_01x01
Connections:
- net GND: now also TH1.1 (Pin_1), TH2.1 (Pin_1), TH3.1 (Pin_1), TH4.1 (Pin_1)
Changed lines of the file:
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@@
     (stroke (width 0) (type default))
   )
-  (polyline (pts (xy 281.94 260.35) (xy 288.29 266.7))
-    (stroke (width 0) (type default))
-  )
   (wire (pts (xy 204.47 78.74) (xy 207.01 78.74))
     (stroke (width 0) (type default))
@@
     (stroke (width 0) (type default))
   )
-  (polyline (pts (xy 288.29 260.35) (xy 281.94 266.7))
-    (stroke (width 0) (type default))
-  )
   (polyline (pts (xy 17.78 13.97) (xy 124.46 13.97))
     (stroke (width 0) (type default))
@@
     (stroke (width 0) (type default))
   )
-  (polyline (pts (xy 288.29 252.73) (xy 281.94 259.08))
-    (stroke (width 0) (type default))
-  )
   (polyline (pts (xy 279.4 123.19) (xy 279.4 212.09))
     (stroke (width 0) (type default))
@@
     (stroke (width 0) (type default))
   )
-  (polyline (pts (xy 281.94 252.73) (xy 288.29 259.08))
-    (stroke (width 0) (type default))
-  )
   (polyline (pts (xy 345.44 72.39) (xy 346.71 72.39))
     (stroke (width 0) (type default))
@@
     )
   )
+  (symbol (lib_id "power:GND") (at 369.57 180.34 270) (unit 1)
+    (in_bom yes) (on_board yes) (dnp no)
+    (property "Reference" "#PWR078" (at 363.22 180.34 0)
+      (effects (font (size 1.27 1.27)) hide)
+    )
+    (property "Value" "GND" (at 365.1758 180.467 0)
+      (effects (font (size 1.27 1.27)) hide)
+    )
+    (property "Footprint" "" (at 369.57 180.34 0)
+      (effects (font (size 1.27 1.27)) hide)
+    )
+    (property "Datasheet" "" (at 369.57 180.34 0)
+      (effects (font (size 1.27 1.27)) hide)
+    )
+    (pin "1")
+    (instances
+      (project "rs-probe"
+        (path "/224768bc-6009-43ba-aa4a-70cbaa15b5a3"
+          (reference "#PWR078") (unit 1)
+        )
+      )
+    )
+  )
   (symbol (lib_id "Device:R_Small") (at 260.35 170.18 180) (unit 1)
     (in_bom yes) (on_board yes) (dnp no) (fields_autoplaced)
@@
     )
   )
+  (symbol (lib_id "Connector_Generic:Conn_01x01") (at 374.65 185.42 0) (unit 1)
+    (in_bom yes) (on_board yes) (dnp no) (fields_autoplaced)
+    (property "Reference" "TH2" (at 377.19 184.15 0)
+      (effects (font (size 1.27 1.27)) (justify left))
+    )
+    (property "Value" "Tooling Hole" (at 377.19 186.69 0)
+      (effects (font (size 1.27 1.27)) (justify left))
+    )
+    (property "Footprint" "" (at 374.65 185.42 0)
+      (effects (font (size 1.27 1.27)) hide)
+    )
+    (property "Datasheet" "~" (at 374.65 185.42 0)
+      (effects (font (size 1.27 1.27)) hide)
+    )
+    (pin "1")
+    (instances
+      (project "rs-probe"
+        (path "/224768bc-6009-43ba-aa4a-70cbaa15b5a3"
+          (reference "TH2") (unit 1)
+        )
+      )
+    )
+  )
   (symbol (lib_id "mosfet:NTZD3155C") (at 201.93 137.16 270) (mirror x) (unit 2)
     (in_bom yes) (on_board yes) (dnp no) (fields_autoplaced)
@@
   )
   (symbol (lib_id "kikit:Tab") (at 285.75 264.16 0) (unit 1)
-    (in_bom no) (on_board no) (dnp no) (fields_autoplaced)
+    (in_bom no) (on_board yes) (dnp no) (fields_autoplaced)
     (property "Reference" "T2" (at 290.83 262.2549 0)
       (effects (font (size 1.27 1.27)) (justify left))
@@
     )
   )
+  (symbol (lib_id "power:GND") (at 369.57 190.5 270) (unit 1)
+    (in_bom yes) (on_board yes) (dnp no)
+    (property "Reference" "#PWR080" (at 363.22 190.5 0)
+      (effects (font (size 1.27 1.27)) hide)
+    )
+    (property "Value" "GND" (at 365.1758 190.627 0)
+      (effects (font (size 1.27 1.27)) hide)
+    )
+    (property "Footprint" "" (at 369.57 190.5 0)
+      (effects (font (size 1.27 1.27)) hide)
+    )
+    (property "Datasheet" "" (at 369.57 190.5 0)
+      (effects (font (size 1.27 1.27)) hide)
+    )
+    (pin "1")
+    (instances
+      (project "rs-probe"
+        (path "/224768bc-6009-43ba-aa4a-70cbaa15b5a3"
+          (reference "#PWR080") (unit 1)
+        )
+      )
+    )
+  )
+  (symbol (lib_id "power:GND") (at 369.57 185.42 270) (unit 1)
+    (in_bom yes) (on_board yes) (dnp no)
+    (property "Reference" "#PWR079" (at 363.22 185.42 0)
+      (effects (font (size 1.27 1.27)) hide)
+    )
+    (property "Value" "GND" (at 365.1758 185.547 0)
+      (effects (font (size 1.27 1.27)) hide)
+    )
+    (property "Footprint" "" (at 369.57 185.42 0)
+      (effects (font (size 1.27 1.27)) hide)
+    )
+    (property "Datasheet" "" (at 369.57 185.42 0)
+      (effects (font (size 1.27 1.27)) hide)
+    )
+    (pin "1")
+    (instances
+      (project "rs-probe"
+        (path "/224768bc-6009-43ba-aa4a-70cbaa15b5a3"
+          (reference "#PWR079") (unit 1)
+        )
+      )
+    )
+  )
   (symbol (lib_id "Regulator_Linear:NCP133AMX100TCG") (at 238.76 168.91 0) (unit 1)
     (in_bom yes) (on_board yes) (dnp no) (fields_autoplaced)
@@
     )
   )
+  (symbol (lib_id "Connector_Generic:Conn_01x01") (at 374.65 180.34 0) (unit 1)
+    (in_bom yes) (on_board yes) (dnp no) (fields_autoplaced)
+    (property "Reference" "TH1" (at 377.19 179.07 0)
+      (effects (font (size 1.27 1.27)) (justify left))
+    )
+    (property "Value" "Tooling Hole" (at 377.19 181.61 0)
+      (effects (font (size 1.27 1.27)) (justify left))
+    )
+    (property "Footprint" "" (at 374.65 180.34 0)
+      (effects (font (size 1.27 1.27)) hide)
+    )
+    (property "Datasheet" "~" (at 374.65 180.34 0)
+      (effects (font (size 1.27 1.27)) hide)
+    )
+    (pin "1")
+    (instances
+      (project "rs-probe"
+        (path "/224768bc-6009-43ba-aa4a-70cbaa15b5a3"
+          (reference "TH1") (unit 1)
+        )
+      )
+    )
+  )
+  (symbol (lib_id "Connector_Generic:Conn_01x01") (at 374.65 190.5 0) (unit 1)
+    (in_bom yes) (on_board yes) (dnp no) (fields_autoplaced)
+    (property "Reference" "TH3" (at 377.19 189.23 0)
+      (effects (font (size 1.27 1.27)) (justify left))
+    )
+    (property "Value" "Tooling Hole" (at 377.19 191.77 0)
+      (effects (font (size 1.27 1.27)) (justify left))
+    )
+    (property "Footprint" "" (at 374.65 190.5 0)
+      (effects (font (size 1.27 1.27)) hide)
+    )
+    (property "Datasheet" "~" (at 374.65 190.5 0)
+      (effects (font (size 1.27 1.27)) hide)
+    )
+    (pin "1")
+    (instances
+      (project "rs-probe"
+        (path "/224768bc-6009-43ba-aa4a-70cbaa15b5a3"
+          (reference "TH3") (unit 1)
+        )
+      )
+    )
+  )
   (symbol (lib_id "power:+3.3V") (at 148.59 90.17 90) (mirror x) (unit 1)
     (in_bom yes) (on_board yes) (dnp no) (fields_autoplaced)
@@
     )
   )
+  (symbol (lib_id "Connector_Generic:Conn_01x01") (at 374.65 195.58 0) (unit 1)
+    (in_bom yes) (on_board yes) (dnp no) (fields_autoplaced)
+    (property "Reference" "TH4" (at 377.19 194.31 0)
+      (effects (font (size 1.27 1.27)) (justify left))
+    )
+    (property "Value" "Tooling Hole" (at 377.19 196.85 0)
+      (effects (font (size 1.27 1.27)) (justify left))
+    )
+    (property "Footprint" "" (at 374.65 195.58 0)
+      (effects (font (size 1.27 1.27)) hide)
+    )
+    (property "Datasheet" "~" (at 374.65 195.58 0)
+      (effects (font (size 1.27 1.27)) hide)
+    )
+    (pin "1")
+    (instances
+      (project "rs-probe"
+        (path "/224768bc-6009-43ba-aa4a-70cbaa15b5a3"
+          (reference "TH4") (unit 1)
+        )
+      )
+    )
+  )
   (symbol (lib_id "Connector_Generic:Conn_01x01") (at 262.89 99.06 0) (unit 1)
     (in_bom no) (on_board yes) (dnp no) (fields_autoplaced)
@@
     )
   )
+  (symbol (lib_id "power:GND") (at 369.57 195.58 270) (unit 1)
+    (in_bom yes) (on_board yes) (dnp no)
+    (property "Reference" "#PWR081" (at 363.22 195.58 0)
+      (effects (font (size 1.27 1.27)) hide)
+    )
+    (property "Value" "GND" (at 365.1758 195.707 0)
+      (effects (font (size 1.27 1.27)) hide)
+    )
+    (property "Footprint" "" (at 369.57 195.58 0)
+      (effects (font (size 1.27 1.27)) hide)
+    )
+    (property "Datasheet" "" (at 369.57 195.58 0)
+      (effects (font (size 1.27 1.27)) hide)
+    )
+    (pin "1")
+    (instances
+      (project "rs-probe"
+        (path "/224768bc-6009-43ba-aa4a-70cbaa15b5a3"
+          (reference "#PWR081") (unit 1)
+        )
+      )
+    )
+  )
   (symbol (lib_id "Device:C_Small") (at 43.18 271.78 0) (unit 1)
     (in_bom yes) (on_board yes) (dnp no)
@@
   )
   (symbol (lib_id "kikit:Tab") (at 285.75 256.54 0) (unit 1)
-    (in_bom no) (on_board no) (dnp no) (fields_autoplaced)
+    (in_bom no) (on_board yes) (dnp no) (fields_autoplaced)
     (property "Reference" "T1" (at 290.83 254.6349 0)
       (effects (font (size 1.27 1.27)) (justify left))
