File: backplane/backplane.kicad_pcb (KiCad board)
At the start: 2 copper layers, 45.8 x 14 mm, 13 parts, among them J5 tag-connect-swd, T1 Tab, T2 Tab

Commit message: final production file
Parts:
- moved SYM1 2.68 mm to (154.5, 96.0)
Other:
- outline, holes or cut-outs redrawn
Changed lines of the file:
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@@
   )
   (footprint "Symbol_Extended:LamudaEE-12.3x7.6mm" (layer "B.Cu")
-    (at 156.6 94.3 180)
+    (at 154.50496 95.978384 180)
     (property "Sheetfile" "rs-probe.kicad_sch")
     (property "Sheetname" "")
@@
       (stroke (width 0) (type solid)) (fill solid) (layer "B.SilkS"))
   )
+  (gr_line (start 159.175 90.375) (end 159.175 92.675)
+    (stroke (width 0.05) (type default)) (layer "Eco1.User"))
+  (gr_line (start 159.175 90.375) (end 161.925 90.375)
+    (stroke (width 0.05) (type default)) (layer "Eco1.User"))
+  (gr_line (start 161.925 90.375) (end 161.925 92.675)
+    (stroke (width 0.05) (type default)) (layer "Eco1.User"))
+  (gr_line (start 159.175 92.675) (end 161.925 92.675)
+    (stroke (width 0.05) (type default)) (layer "Eco1.User"))
   (gr_circle (center 165.5 87.5) (end 166.076 87.5)
     (stroke (width 0.05) (type default)) (fill none) (layer "Edge.Cuts"))
@@
   (gr_line (start 175.8 86.5) (end 175.8 87.5)
     (stroke (width 0.1) (type solid)) (layer "Edge.Cuts"))
+  (gr_line (start 162.025 90.375) (end 162.025 92.675)
+    (stroke (width 0.05) (type default)) (layer "Edge.Cuts"))
   (gr_circle (center 137.5 93) (end 138.076 93)
     (stroke (width 0.05) (type default)) (fill none) (layer "Edge.Cuts"))
@@
   (gr_line (start 175.3 98) (end 168.7 98)
     (stroke (width 0.1) (type solid)) (layer "Edge.Cuts"))
+  (gr_line (start 159.175 92.775) (end 161.925 92.775)
+    (stroke (width 0.05) (type default)) (layer "Edge.Cuts"))
+  (gr_line (start 159.175 92.775) (end 159.075 92.675)
+    (stroke (width 0.05) (type default)) (layer "Edge.Cuts"))
+  (gr_line (start 161.925 92.775) (end 162.025 92.675)
+    (stroke (width 0.05) (type default)) (layer "Edge.Cuts"))
   (gr_line (start 146.4 98) (end 146.4 99.5)
     (stroke (width 0.1) (type solid)) (layer "Edge.Cuts"))
   (gr_line (start 175.3 86) (end 175.8 86.5)
     (stroke (width 0.1) (type solid)) (layer "Edge.Cuts"))
+  (gr_line (start 159.075 90.375) (end 159.175 90.275)
+    (stroke (width 0.05) (type default)) (layer "Edge.Cuts"))
   (gr_line (start 137.2 97.5) (end 136.7 98)
     (stroke (width 0.1) (type solid)) (layer "Edge.Cuts"))
+  (gr_line (start 159.175 90.275) (end 161.925 90.275)
+    (stroke (width 0.05) (type default)) (layer "Edge.Cuts"))
   (gr_line (start 132.5 97.5) (end 132 97)
     (stroke (width 0.1) (type solid)) (layer "Edge.Cuts"))
   (gr_line (start 175.8 87.5) (end 175.3 88)
     (stroke (width 0.1) (type solid)) (layer "Edge.Cuts"))
+  (gr_line (start 161.925 90.275) (end 162.025 90.375)
+    (stroke (width 0.05) (type default)) (layer "Edge.Cuts"))
   (gr_line (start 132.5 99.5) (end 132.5 97.5)
     (stroke (width 0.1) (type solid)) (layer "Edge.Cuts"))
@@
   (gr_line (start 132 89) (end 130 89)
     (stroke (width 0.1) (type solid)) (layer "Edge.Cuts"))
+  (gr_line (start 159.075 90.375) (end 159.075 92.675)
+    (stroke (width 0.05) (type default)) (layer "Edge.Cuts"))
   (gr_line (start 135.6 90.7) (end 135.1 90.2)
     (stroke (width 0.1) (type solid)) (layer "Edge.Cuts"))
@@
     (effects (font (size 0.8 0.8) (thickness 0.153) bold) (justify left bottom))
   )
-  (gr_text "Rusty-Probe BackPlane" (at 146.9 90.9) (layer "F.SilkS")
+  (gr_text "Rusty-Probe BackPlane" (at 147.1 89.8) (layer "F.SilkS")
     (effects (font (size 1 1) (thickness 0.16)) (justify left bottom))
   )
